File: Hardware/Electronics/Music Player.kicad_sch (KiCad schematic)
At the start: 33 parts, among them J1 USB_B_Micro, U2 W25Q128JVS, U3 APS6404L-3SQRx-SN, U4 USBLC6-2SC6, Y1 ABM8-272-T3

Commit message: Added schematic PDF and schematic sheet information
Other:
- title: (none) -> Microcontroller
Changed lines of the file:
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@@
 	(generator_version "9.0")
 	(paper "A3")
+	(title_block
+		(title "Microcontroller")
+		(date "2025-12-05")
+		(rev "0")
+	)
 	(rectangle
 		(start 95.25 17.78)

Commit message: Added SD card, and started adding power management
Parts:
- added C21: 100nF, symbol Device:C
- added C22: 1nF, symbol Device:C
- added C23: 47nF, symbol Device:C_Small
- added C24, C25, C26: 10uF, symbol Device:C_Small
- added F1: 2A, symbol Device:Fuse
- added J2: Micro_SD_Card_Det1, symbol Connector:Micro_SD_Card_Det1
- added J3: Conn_01x02, Connector_JST:JST_EH_B2B-EH-A_1x02_P2.50mm_Vertical, symbol Connector_Generic:Conn_01x02
- added L2: 2.2uH, symbol Device:L
- added Q1: SI231DS, Package_TO_SOT_SMD:SOT-23, symbol Transistor_FET:Q_NMOS_GSD
- added Q2: AO3407A, Package_TO_SOT_SMD:SOT-23, symbol Transistor_FET:Q_PMOS_GSD
- added R10, R11, R12, R13, R9: 47kR, symbol Device:R_Small
- added R14: 262kR, symbol Device:R
- added R15: 100kR, symbol Device:R
- added R16: 10kR, symbol Device:R
- added R17: 10kR, symbol Device:R_Small
- added R18: 333R, symbol Device:R
- added R7, R8: 1kR, symbol Device:R_Small
- added SW1, SW2: SW_SPST, symbol Switch:SW_SPST
- added U5: BQ24195, Package_DFN_QFN:VQFN-24-1EP_4x4mm_P0.5mm_EP2.5x2.5mm_ThermalVias, symbol Symbol Library:BQ24195
Connections:
- net +3V3: now also C21.1, J2.4 (VDD), R10.1, R11.1, R12.1, R13.1, R9.1
- net +5V: now also Q2.3 (D), R14.1
- net GND: now also C21.2, C24.2, C25.2, C26.2, J2.10 (SHIELD), J2.6 (VSS), J3.1 (Pin_1), Q1.2 (S), R15.2, R17.2, R18.2, R7.2, R8.2, U5.17 (PGND), U5.18 (PGND), U5.8 (OTG)
- net QSPI_SS: now also SW2.2 (B)
- net USB_D+: now also U5.2 (D+)
- net USB_D-: now also U5.3 (D-)
- net CHRG_CE: now reaches U1.19 (GPIO15)
- net CHRG_CE: now also R17.1, U5.9 (~{CE})
- net at U1.26 (RUN): now also SW1.2 (B)
- net CHRG_SDA: now reaches U1.27 (GPIO16)
- net CHRG_SDA: now also U5.6 (SDA)
- net CHRG_SCL: now reaches U1.28 (GPIO17)
- net CHRG_SCL: now also U5.5 (SCL)
- net CHRG_INT: now reaches U1.29 (GPIO18)
- net CHRG_INT: now also U5.7 (INT)
- net SDIO_DET: now reaches U1.31 (GPIO19)
- net SDIO_DET: now also J2.9 (DET)
- net SDIO_CLK: now reaches U1.32 (GPIO20)
- net SDIO_CLK: now also J2.5 (CLK)
- net SDIO_CMD: now reaches U1.33 (GPIO21)
- net SDIO_CMD: now also J2.3 (CMD), R13.2
- net SDIO_DAT3: now reaches U1.34 (GPIO22)
- net SDIO_DAT3: now also J2.2 (DAT3/CD), R12.2
- net SDIO_DAT2: now reaches U1.35 (GPIO23)
- net SDIO_DAT2: now also J2.1 (DAT2), R11.2
- net SDIO_DAT1: now reaches U1.36 (GPIO24)
- net SDIO_DAT1: now also J2.8 (DAT1), R10.2
- net SDIO_DAT0: now reaches U1.37 (GPIO25)
- net SDIO_DAT0: now also J2.7 (DAT0), R9.2
- net BATT_MON: now reaches U1.40 (GPIO26_ADC0)
- new net: C23.1, L2.1, U5.19 (SW), U5.20 (SW)
- new net: C24.1, C25.1, L2.2, U5.15 (SYS), U5.16 (SYS)
- new net: C22.1, Q2.2 (S), R16.2, U5.1 (VBUS), U5.24 (VBUS)
- new net: C22.2, Q1.3 (D), Q2.1 (G), R16.1
- new net: Q1.1 (G), R14.2, R15.1
- new net: R18.1, U5.10 (ILIM)
- new net: F1.1, U5.13 (BAT), U5.14 (BAT)
- new net: C23.2, U5.21 (BTST)
- new net: C26.1, U5.22 (RGEN)
- new net: R8.1, SW2.1 (A)
- new net: R7.1, SW1.1 (A)
- new net: F1.2, J3.2 (Pin_2)
- no-connect marks 1 -> 2
Other:
- note added: "ADD LED"
- note added: "ADD THERMAL PROTECTION"
- note added: "Micro SD Card"
- note added: "POWER MANAGEMENT"
- note added: "TO DO: Finish Power Management (3.3V Voltage Regulator & thermal protection) Buttons (interface and power) DAC & headphone output Audio bluetooth module (feasycom bt1058) 4G module"
- moved on the sheet: R5, R6, U1
